File: MobileAdapter.kicad_pcb (KiCad board)
At the start: 4 copper layers, 51.5 x 50 mm, 36 parts, among them J1 VID0, J2 VID1, J3 VID2, J4 VID3

Commit message: Trace and Silk fix
Routing:
- net PLL1: track 0.90 -> 27.6 mm, vias 1 -> 2
- net SMI: track 25.9 -> 26.6 mm
Other:
- board text added: "1"
- board text added: "2"
- board text added: "3"
